File: CanoKey NFC-A v2/PCB/Main.sch (KiCad schematic (older format))
At the start: 31 parts, among them J1 USB_A_PCB, U1 FM11NC08S, U2 USBLC6-2SC6, U3 STM32L432KCUx, U4 AP7331-33SNG-7

Commit message: add Manufacturing File
Parts:
- C1: Dielectric (none) -> x7r; Field5 25v -> (none); Voltage (none) -> 50v
- C2, C3, C4: Dielectric (none) -> x7r; Field5 25v -> (none); LCSC (none) -> C14663; Voltage (none) -> 50v
- C5, C6: Dielectric (none) -> x5r; Field5 25v -> (none); LCSC (none) -> C15849; Voltage (none) -> 25v
- D1, D3: LCSC (none) -> C282367
- D2: Field4 C409780 -> (none); LCSC (none) -> C409780
- R1, R2, R4: Field5 5% -> (none); LCSC (none) -> C23345; Tolerance (none) -> 5%
- R10, R11, R12, R6, R9: Field5 5% -> (none); Tolerance (none) -> 5%
- R3, R5, R8: Field5 5% -> (none); LCSC (none) -> C4190; Tolerance (none) -> 5%
- R7: Field5 5% -> (none); LCSC (none) -> C23196; Tolerance (none) -> 5%
- U1: Field4 C182885 -> (none); LCSC (none) -> C182885
- U2: LCSC (none) -> C7519
- U3: Field4 C94784 -> (none); LCSC (none) -> C94784
- U4: Field4 C150446 -> (none); LCSC (none) -> C150446
Changed lines of the file:
@@
 F 2 "Package_DFN_QFN:QFN-32-1EP_5x5mm_P0.5mm_EP3.45x3.45mm" H 5600 1800 50  0001 R CNN
 F 3 "http://www.st.com/st-web-ui/static/active/en/resource/technical/document/datasheet/DM00257205.pdf" H 6000 2700 50  0001 C CNN
-F 4 "C94784" H 6000 2700 50  0001 C CNN "Field4"
+F 4 "C94784" H 6000 2700 50  0001 C CNN "LCSC"
 	1    6000 2700
 	1    0    0    -1
@@
 F 2 "LED_SMD:LED_RGB_5050-6" H 6050 5350 50  0001 C CNN
 F 3 "https://datasheet.lcsc.com/szlcsc/1912111437_MEIHUA-MHP5050RGBDT_C409780.pdf" H 6050 5650 50  0001 C CNN
-F 4 "C409780" H 6050 5700 50  0001 C CNN "Field4"
+F 4 "C409780" H 6050 5700 50  0001 C CNN "LCSC"
 	1    6050 5700
 	-1   0    0    -1
@@
 F 2 "Capacitor_SMD:C_0603_1608Metric" H 1500 3750 50  0001 C CNN
 F 3 "~" H 1500 3750 50  0001 C CNN
-F 4 "" H 1500 3750 50  0001 C CNN "Field4"
-F 5 "25v" H 1500 3750 50  0001 C CNN "Field5"
-F 6 "" H 1500 3750 50  0001 C CNN "Field6"
+F 4 "~" H 1500 3750 50  0001 C CNN "LCSC"
+F 5 "50v" H 1500 3750 50  0001 C CNN "Voltage"
+F 6 "x7r" H 1500 3750 50  0001 C CNN "Dielectric"
 	1    1500 3750
 	1    0    0    -1
@@
 F 2 "Package_DFN_QFN:DFN-10-1EP_3x3mm_P0.5mm_EP1.55x2.48mm" H 2500 3000 50  0001 C CIN
 F 3 "https://datasheet.lcsc.com/szlcsc/Shanghai-Fudan-Microelectronics-FM11NC08S_C182885.pdf" H 1950 3550 50  0001 C CNN
-F 4 "C182885" H 2500 3700 50  0001 C CNN "Field4"
+F 4 "C182885" H 2500 3700 50  0001 C CNN "LCSC"
 	1    2500 3700
 	1    0    0    -1
@@
 F 2 "Package_TO_SOT_SMD:SOT-23-6" H 2400 6250 50  0001 C CNN
 F 3 "https://www.st.com/resource/en/datasheet/usblc6-2.pdf" H 2600 7100 50  0001 C CNN
+F 4 "C7519" V 2400 6750 50  0001 C CNN "LCSC"
 	1    2400 6750
 	0    1    -1   0
@@
 F 2 "Resistor_SMD:R_0603_1608Metric" H 6350 6100 50  0001 C CNN
 F 3 "~" H 6350 6100 50  0001 C CNN
-F 4 "" H 6350 6100 50  0001 C CNN "Field4"
-F 5 "5%" H 6350 6100 50  0001 C CNN "Field5"
+F 4 "C4190" H 6350 6100 50  0001 C CNN "LCSC"
+F 5 "5%" H 6350 6100 50  0001 C CNN "Tolerance"
 	1    6350 6100
 	-1   0    0    -1
@@
 F 2 "Resistor_SMD:R_0603_1608Metric" H 9150 1700 50  0001 C CNN
 F 3 "~" H 9150 1700 50  0001 C CNN
-F 4 "" H 9150 1700 50  0001 C CNN "Field4"
-F 5 "5%" H 9150 1700 50  0001 C CNN "Field5"
+F 4 "C23196" H 9150 1700 50  0001 C CNN "LCSC"
+F 5 "5%" H 9150 1700 50  0001 C CNN "Tolerance"
 	1    9150 1700
 	1    0    0    -1
@@
 F 2 "Resistor_SMD:R_0603_1608Metric" H 6750 6100 50  0001 C CNN
 F 3 "~" H 6750 6100 50  0001 C CNN
-F 4 "" H 6750 6100 50  0001 C CNN "Field4"
-F 5 "5%" H 6750 6100 50  0001 C CNN "Field5"
+F 4 "C4190" H 6750 6100 50  0001 C CNN "LCSC"
+F 5 "5%" H 6750 6100 50  0001 C CNN "Tolerance"
 	1    6750 6100
 	-1   0    0    -1
@@
 F 2 "Resistor_SMD:R_0603_1608Metric" H 6550 6100 50  0001 C CNN
 F 3 "~" H 6550 6100 50  0001 C CNN
-F 4 "" H 6550 6100 50  0001 C CNN "Field4"
-F 5 "5%" H 6550 6100 50  0001 C CNN "Field5"
+F 4 "C4190" H 6550 6100 50  0001 C CNN "LCSC"
+F 5 "5%" H 6550 6100 50  0001 C CNN "Tolerance"
 	1    6550 6100
 	-1   0    0    -1
@@
 F 2 "Capacitor_SMD:C_0603_1608Metric" H 3400 1700 50  0001 C CNN
 F 3 "~" H 3400 1700 50  0001 C CNN
-F 4 "" H 3400 1700 50  0001 C CNN "Field4"
-F 5 "25v" H 3400 1700 50  0001 C CNN "Field5"
-F 6 "" H 3400 1700 50  0001 C CNN "Field6"
+F 4 "C14663" H 3400 1700 50  0001 C CNN "LCSC"
+F 5 "50v" H 3400 1700 50  0001 C CNN "Voltage"
+F 6 "x7r" H 3400 1700 50  0001 C CNN "Dielectric"
 	1    3400 1700
 	1    0    0    -1
@@
 F 2 "Capacitor_SMD:C_0603_1608Metric" H 3000 1700 50  0001 C CNN
 F 3 "~" H 3000 1700 50  0001 C CNN
-F 4 "" H 3000 1700 50  0001 C CNN "Field4"
-F 5 "25v" H 3000 1700 50  0001 C CNN "Field5"
-F 6 "" H 3000 1700 50  0001 C CNN "Field6"
+F 4 "C14663" H 3000 1700 50  0001 C CNN "LCSC"
+F 5 "50v" H 3000 1700 50  0001 C CNN "Voltage"
+F 6 "x7r" H 3000 1700 50  0001 C CNN "Dielectric"
 	1    3000 1700
 	1    0    0    -1
@@
 F 2 "Capacitor_SMD:C_0603_1608Metric" H 3800 1700 50  0001 C CNN
 F 3 "~" H 3800 1700 50  0001 C CNN
-F 4 "" H 3800 1700 50  0001 C CNN "Field4"
-F 5 "25v" H 3800 1700 50  0001 C CNN "Field5"
-F 6 "" H 3800 1700 50  0001 C CNN "Field6"
+F 4 "C14663" H 3800 1700 50  0001 C CNN "LCSC"
+F 5 "50v" H 3800 1700 50  0001 C CNN "Voltage"
+F 6 "x7r" H 3800 1700 50  0001 C CNN "Dielectric"
 	1    3800 1700
 	1    0    0    -1
@@
 F 2 "MAS_Package_nostd:UDFN-6-1EP_2x2mm_P0.65mm_EP0.9x1.65mm" H 1700 1925 50  0001 C CIN
 F 3 "" H 1700 1600 50  0001 C CNN
-F 4 "C150446" H 1700 1600 50  0001 C CNN "Field4"
+F 4 "C150446" H 1700 1600 50  0001 C CNN "LCSC"
 	1    1700 1600
 	1    0    0    -1
@@
 F 2 "Capacitor_SMD:C_0603_1608Metric" H 1000 1700 50  0001 C CNN
 F 3 "~" H 1000 1700 50  0001 C CNN
-F 4 "" H 1000 1700 50  0001 C CNN "Field4"
-F 5 "25v" H 1000 1700 50  0001 C CNN "Field5"
-F 6 "" H 1000 1700 50  0001 C CNN "Field6"
+F 4 "C15849" H 1000 1700 50  0001 C CNN "LCSC"
+F 5 "25v" H 1000 1700 50  0001 C CNN "Voltage"
+F 6 "x5r" H 1000 1700 50  0001 C CNN "Dielectric"
 	1    1000 1700
 	1    0    0    -1
@@
 F 2 "Capacitor_SMD:C_0603_1608Metric" H 2500 1700 50  0001 C CNN
 F 3 "~" H 2500 1700 50  0001 C CNN
-F 4 "" H 2500 1700 50  0001 C CNN "Field4"
-F 5 "25v" H 2500 1700 50  0001 C CNN "Field5"
-F 6 "" H 2500 1700 50  0001 C CNN "Field6"
+F 4 "C15849" H 2500 1700 50  0001 C CNN "LCSC"
+F 5 "25v" H 2500 1700 50  0001 C CNN "Voltage"
+F 6 "x5r" H 2500 1700 50  0001 C CNN "Dielectric"
 	1    2500 1700
 	-1   0    0    -1
@@
 F 2 "Resistor_SMD:R_0603_1608Metric" H 9150 1300 50  0001 C CNN
 F 3 "~" H 9150 1300 50  0001 C CNN
-F 4 "" H 9150 1300 50  0001 C CNN "Field4"
-F 5 "5%" H 9150 1300 50  0001 C CNN "Field5"
+F 4 "" H 9150 1300 50  0001 C CNN "LCSC"
+F 5 "5%" H 9150 1300 50  0001 C CNN "Tolerance"
 	1    9150 1300
 	1    0    0    -1
@@
 F 2 "Resistor_SMD:R_0603_1608Metric" H 2950 6250 50  0001 C CNN
 F 3 "~" H 2950 6250 50  0001 C CNN
-F 4 "" H 2950 6250 50  0001 C CNN "Field4"
-F 5 "5%" H 2950 6250 50  0001 C CNN "Field5"
+F 4 "C23345" H 2950 6250 50  0001 C CNN "LCSC"
+F 5 "5%" H 2950 6250 50  0001 C CNN "Tolerance"
 	1    2950 6250
 	0    1    -1   0
@@
 F 2 "Resistor_SMD:R_0603_1608Metric" H 2950 7250 50  0001 C CNN
 F 3 "~" H 2950 7250 50  0001 C CNN
-F 4 "" H 2950 7250 50  0001 C CNN "Field4"
-F 5 "5%" H 2950 7250 50  0001 C CNN "Field5"
+F 4 "C23345" H 2950 7250 50  0001 C CNN "LCSC"
+F 5 "5%" H 2950 7250 50  0001 C CNN "Tolerance"
 	1    2950 7250
 	0    1    -1   0
@@
 F 2 "Resistor_SMD:R_0603_1608Metric" H 8950 1500 50  0001 C CNN
 F 3 "~" H 8950 1500 50  0001 C CNN
-F 4 "" H 8950 1500 50  0001 C CNN "Field4"
-F 5 "5%" H 8950 1500 50  0001 C CNN "Field5"
+F 4 "C23345" H 8950 1500 50  0001 C CNN "LCSC"
+F 5 "5%" H 8950 1500 50  0001 C CNN "Tolerance"
 	1    8950 1500
 	0    -1   -1   0
@@
 F 2 "Package_TO_SOT_SMD:SOT-363_SC-70-6" V 950 3550 50  0001 L CNN
 F 3 "https://assets.nexperia.com/documents/data-sheet/BAT54XY.pdf" V 1350 4030 50  0001 C CNN
+F 4 "C282367" V 1350 4550 50  0001 C CNN "LCSC"
 	1    1350 4550
 	0    -1   -1   0
@@
 F 2 "Package_TO_SOT_SMD:SOT-363_SC-70-6" V 9200 850 50  0001 L CNN
 F 3 "https://assets.nexperia.com/documents/data-sheet/BAT54XY.pdf" V 9600 1330 50  0001 C CNN
+F 4 "C282367" V 9600 1850 50  0001 C CNN "LCSC"
 	1    9600 1850
 	0    -1   -1   0
@@
 F 2 "Resistor_SMD:R_0603_1608Metric" H 9650 5350 50  0001 C CNN
 F 3 "~" H 9650 5350 50  0001 C CNN
-F 4 "" H 9650 5350 50  0001 C CNN "Field4"
-F 5 "5%" H 9650 5350 50  0001 C CNN "Field5"
+F 4 "" H 9650 5350 50  0001 C CNN "LCSC"
+F 5 "5%" H 9650 5350 50  0001 C CNN "Tolerance"
 	1    9650 5350
 	0    1    -1   0
@@
 F 2 "Resistor_SMD:R_0603_1608Metric" H 9650 5500 50  0001 C CNN
 F 3 "~" H 9650 5500 50  0001 C CNN
-F 4 "" H 9650 5500 50  0001 C CNN "Field4"
-F 5 "5%" H 9650 5500 50  0001 C CNN "Field5"
+F 4 "" H 9650 5500 50  0001 C CNN "LCSC"
+F 5 "5%" H 9650 5500 50  0001 C CNN "Tolerance"
 	1    9650 5500
 	0    1    -1   0
@@
 F 2 "Resistor_SMD:R_0603_1608Metric" H 9650 5650 50  0001 C CNN
 F 3 "~" H 9650 5650 50  0001 C CNN
-F 4 "" H 9650 5650 50  0001 C CNN "Field4"
-F 5 "5%" H 9650 5650 50  0001 C CNN "Field5"
+F 4 "" H 9650 5650 50  0001 C CNN "LCSC"
+F 5 "5%" H 9650 5650 50  0001 C CNN "Tolerance"
 	1    9650 5650
 	0    1    -1   0
@@
 F 2 "Resistor_SMD:R_0603_1608Metric" H 9650 5800 50  0001 C CNN
 F 3 "~" H 9650 5800 50  0001 C CNN
-F 4 "" H 9650 5800 50  0001 C CNN "Field4"
-F 5 "5%" H 9650 5800 50  0001 C CNN "Field5"
+F 4 "" H 9650 5800 50  0001 C CNN "LCSC"
+F 5 "5%" H 9650 5800 50  0001 C CNN "Tolerance"
 	1    9650 5800
 	0    1    -1   0
